Commit message: Forgot to add clock

File: src/first_robot/robot_description/first_robot.urdf.xacro (robot description, xacro)
@@ -4,5 +4,8 @@
     <xacro:include filename="$(find first_robot_freecad)/urdf/FirstRobot.urdf" />
     <!-- Add ROS2 Control to the wheel joints -->
-    <ros2_control name="magni" type="system">
+    <ros2_control name="first_robot" type="system">
+        <hardware>
+            <plugin>ign_ros2_control/IgnitionSystem</plugin>
+        </hardware>
         <joint name="left_wheel_joint">
             <command_interface name="velocity">
@@ -24,16 +27,4 @@
         </joint>
     </ros2_control>
-    <!-- Setup plugins for control -->
-    <gazebo>
-        <plugin filename="ign_ros2_control-system" name="ign_ros2_control::IgnitionROS2ControlPlugin">
-            <controller_manager_prefix_node_name>/krytn</controller_manager_prefix_node_name>
-            <ros>
-                <remapping>diff_drive_base_controller/odometry:=odom</remapping>
-                <remapping>diff_drive_base_controller/tf_odometry:=tf</remapping>
-                <remapping>diff_drive_base_controller/cmd_vel_unstamped:=cmd_vel</remapping>
-            </ros>
-            <parameters>$(find first_robot)/config/diffdrive_control.yaml</parameters>
-        </plugin>
-    </gazebo>
     <!-- Adding a lidar sensor to the base link, feel free to change the reference to the name of a link that you want the lidar to be in -->
     <gazebo reference="base_link">
@@ -67,3 +58,23 @@
         </sensor>
     </gazebo>
+    <!-- Add a dummy base_footprint link to remove error messages about it. -->
+    <link name="base_footprint"/>
+    <joint name="base_fp_link" type="fixed">
+        <parent link="base_footprint" />
+        <child link="base_link" />
+    </joint>
+    <!-- Setup plugins for control and sensors -->
+    <gazebo>
+        <plugin filename="ign_ros2_control-system" name="ign_ros2_control::IgnitionROS2ControlPlugin">
+            <ros>
+                <remapping>diff_drive_base_controller/odometry:=odom</remapping>
+                <remapping>diff_drive_base_controller/tf_odometry:=tf</remapping>
+                <remapping>diff_drive_base_controller/cmd_vel_unstamped:=cmd_vel</remapping>
+            </ros>
+            <parameters>$(find first_robot)/config/diffdrive_control.yaml</parameters>
+        </plugin>
+        <plugin filename="ignition-gazebo-sensors-system" name="ignition::gazebo::systems::Sensors">
+            <render_engine>ogre2</render_engine>
+        </plugin>
+    </gazebo>
 </robot>

Commit message: adjusting freecad design and gazebo scripts

File: src/first_robot/robot_description/first_robot.urdf.xacro (robot description, xacro)
@@ -78,3 +78,95 @@
         </plugin>
     </gazebo>
+    <!-- Increase friction of wheels so they don't slip as much -->
+    <gazebo reference="left_wheel">
+        <collision>
+            <surface>
+                <friction>
+                    <ode>
+                        <mu>1.0</mu>
+                        <mu2>1.0</mu2>
+                        <fdir1>0 0 1</fdir1>
+                        <slip1>0.0</slip1>
+                        <slip2>0.0</slip2>
+                        <min_depth>0.001</min_depth>
+                        <kp>1e8</kp>
+                    </ode>
+                </friction>
+            </surface>
+        </collision>
+    </gazebo>
+    <gazebo reference="right_wheel">
+        <collision>
+            <surface>
+                <friction>
+                    <ode>
+                        <mu>10000</mu>
+                        <mu2>10000</mu2>
+                        <fdir1>0 0 1</fdir1>
+                        <slip1>0.001</slip1>
+                        <slip2>0.001</slip2>
+                        <min_depth>0.001</min_depth>
+                        <kp>1e8</kp>
+                    </ode>
+                    <bullet>
+                        <friction>1</friction>
+                        <friction2>1</friction2>
+                        <rolling_friction>0.1</rolling_friction>
+                    </bullet>
+                </friction>
+            </surface>
+        </collision>
+    </gazebo>
+    <!-- Reduce friction of base link so it will slide -->
+    <gazebo reference="base_link">
+        <collision>
+            <surface>
+                <contact>
+                    <min_depth>0.0001</min_depth>
+                </contact>
+                <friction>
+                    <ode>
+                        <mu>0.01</mu>
+                        <mu1>0.01</mu1>
+                        <mu2>0.01</mu2>
+                        <slip1>0.01</slip1>
+                        <slip2>0.01</slip2>
+                        <kp>1e-1</kp>
+                        <kd>1e-1</kd>
+                    </ode>
+                    <bullet>
+                        <friction>1</friction>
+                        <friction2>1</friction2>
+                        <rolling_friction>0.1</rolling_friction>
+                    </bullet>
+                </friction>
+            </surface>
+        </collision>
+    </gazebo>
+    <!-- Reduce friction of base link so it will slide -->
+    <gazebo reference="caster_wheel">
+        <collision>
+            <surface>
+                <contact>
+                    <min_depth>0.0001</min_depth>
+                </contact>
+                <friction>
+                    <ode>
+                        <mu>0.01</mu>
+                        <mu1>0.01</mu1>
+                        <mu2>0.01</mu2>
+                        <slip1>0.01</slip1>
+                        <slip2>0.01</slip2>
+                        <kp>1e-1</kp>
+                        <kd>1e-1</kd>
+                    </ode>
+                    <bullet>
+                        <friction>1</friction>
+                        <friction2>1</friction2>
+                        <rolling_friction>0.1</rolling_friction>
+                    </bullet>
+                </friction>
+            </surface>
+        </collision>
+    </gazebo>
 </robot>

File: src/first_robot_freecad/urdf/FirstRobot.urdf (robot description, URDF)
Before this commit: robot Robot, 3 links, 2 joints
Links:
- added link caster_wheel, mass 0.0; collision sphere radius=0.04; visual sphere radius=0.04
Joints:
- added joint caster_wheel_joint: type fixed, parent base_link, child caster_wheel, origin xyz=-0.25 0.0 -0.04 rpy=0.0 -0.0 0.0
- joint right_wheel_joint: origin xyz=0.0 -0.12 0.0 rpy=1.5707963267948966 -0.0 0.0 -> xyz=0.0 -0.12 0.0 rpy=-1.5707963267948966 0.0 0.0
