Commit message: Adjusting gazebo.launch.py and others to load

File: src/bar_examples/magni_description/urdf/magni.urdf.xacro (robot description, xacro)
@@ -3,5 +3,5 @@
   <xacro:property name="wheel_r" value="0.1" />
   <xacro:property name="wheel_xpos" value="0.11" />
-  <xacro:include filename="$(find krytn)/robot_description/magni/inertial.xacro" />
+  <xacro:include filename="$(find magni_description)/urdf/inertial.xacro" />
   <xacro:macro name="low_friction">
     <collision>
@@ -44,5 +44,5 @@
       <origin xyz="${-wheel_xpos} 0 ${-wheel_r+0.071}" rpy="0 0 0" />
       <geometry>
-        <mesh filename="file://$(find krytn)/robot_description/magni/meshes/magni_body.dae" />
+        <mesh filename="file://$(find magni_description)/meshes/magni_body.dae" />
       </geometry>
     </visual>
@@ -90,5 +90,5 @@
         <origin xyz="${-0.071*reflect} 0 0" rpy="0 ${(reflect-1)*pi/2} 0" />
         <geometry>
-          <mesh filename="file://$(find krytn)/robot_description/magni/meshes/front_wheel.dae" />
+          <mesh filename="file://$(find magni_description)/meshes/front_wheel.dae" />
         </geometry>
       </visual>
@@ -125,5 +125,5 @@
         <origin xyz="-0.25 ${reflect*0.169} 0" rpy="0 0 ${pi}" />
         <geometry>
-          <mesh filename="file://$(find krytn)/robot_description/magni/meshes/caster_wheel.dae" />
+          <mesh filename="file://$(find magni_description)/meshes/caster_wheel.dae" />
         </geometry>
       </visual>

Commit message: Getting teleop working

File: src/bar_examples/magni_description/urdf/magni.urdf.xacro (robot description, xacro)
@@ -8,11 +8,13 @@
       <surface>
         <friction>
-          <mu>0.1</mu>
-          <mu1>0.1</mu1>
-          <mu2>0.1</mu2>
-          <slip1>0</slip1>
-          <slip2>0</slip2>
+          <ode>
+            <mu>0.1</mu>
+            <mu2>0.1</mu2>
+            <slip1>0</slip1>
+            <slip2>0</slip2>
+          </ode>
         </friction>
       </surface>
+      <max_contacts>1</max_contacts>
     </collision>
   </xacro:macro>
@@ -30,4 +32,5 @@
         </friction>
       </surface>
+      <max_contacts>1</max_contacts>
     </collision>
   </xacro:macro>

File: src/bar_examples/sensors/realsense_d435/realsense.urdf.xacro (robot description, xacro)
@@ -1,58 +1,43 @@
 <robot name="sensor_d435"
     xmlns:xacro="http://ros.org/wiki/xacro">
-    <xacro:macro name="realsense" param="base_link">
+    <xacro:macro name="realsense" params="world_link_name *origin">
         <link name="realsense_link">
-            <inertial>
-                <mass>0.0615752</mass>
-                <inertia>
-                    <ixx>9.108e-05</ixx>
-                    <ixy>0</ixy>
-                    <ixz>0</ixz>
-                    <iyy>2.51e-06</iyy>
-                    <iyz>0</iyz>
-                    <izz>8.931e-05</izz>
-                </inertia>
-                <pose frame=''>0 0 0 0 -0 0</pose>
-            </inertial>
+            <xacro:box_inertial x="0.02" y="0.1" z="0.01" mass="0.06"/>
             <collision name="collision">
                 <geometry>
-                    <mesh>
-                        <uri>package://sensors/realsense_d435/meshes/realsense.dae</uri>
-                    </mesh>
+                    <mesh filename="package://sensors/realsense_d435/meshes/realsense.dae" />
                 </geometry>
             </collision>
             <visual name= "visual">
+                <origin rpy="0 0 ${pi/2}"/>
                 <geometry>
-                    <mesh>
-                        <uri>package://sensors/realsense_d435/meshes/realsense.dae</uri>
-                        <submesh>
-                            <name>RealSense</name>
-                            <center>false</center>
-                        </submesh>
-                    </mesh>
+                    <mesh filename="package://sensors/realsense_d435/meshes/realsense.dae"/>
                 </geometry>
-                <material>
-                    <diffuse>1.0 1.0 1.0</diffuse>
-                    <specular>1.0 1.0 1.0</specular>
-                    <pbr>
-                        <metal>
-                            <albedo_map>package://sensors/realsense_d435/materials/textures/RealSense_Albedo.png</albedo_map>
-                            <normal_map>package://sensors/realsense_d435/materials/textures/RealSense_Normal.png</normal_map>
-                            <metalness_map>package://sensors/realsense_d435/materials/textures/RealSense_Metalness.png</metalness_map>
-                            <roughness_map>package://sensors/realsense_d435/materials/textures/RealSense_Roughness.png</roughness_map>
-                        </metal>
-                    </pbr>
-                    <!-- fallback to script if no PBR support-->
-                    <script>
-                        <uri>package://sensors/realsense_d435/materials/scripts/</uri>
-                        <uri>package://sensors/realsense_d435/materials/textures/</uri>
-                        <name>UrbanTile/RealSense_Diffuse</name>
-                    </script>
-                </material>
+                <gazebo>
+                    <material>
+                        <diffuse>1.0 1.0 1.0</diffuse>
+                        <specular>1.0 1.0 1.0</specular>
+                        <pbr>
+                            <metal>
+                                <albedo_map>package://sensors/realsense_d435/materials/textures/RealSense_Albedo.png</albedo_map>
+                                <normal_map>package://sensors/realsense_d435/materials/textures/RealSense_Normal.png</normal_map>
+                                <metalness_map>package://sensors/realsense_d435/materials/textures/RealSense_Metalness.png</metalness_map>
+                                <roughness_map>package://sensors/realsense_d435/materials/textures/RealSense_Roughness.png</roughness_map>
+                            </metal>
+                        </pbr>
+                        <!-- fallback to script if no PBR support-->
+                        <script>
+                            <uri>package://sensors/realsense_d435/materials/scripts/</uri>
+                            <uri>package://sensors/realsense_d435/materials/textures/</uri>
+                            <name>UrbanTile/RealSense_Diffuse</name>
+                        </script>
+                    </material>
+                </gazebo>
             </visual>
         </link>
         <gazebo reference="realsense_link">
             <sensor name="realsense_d435" type="rgbd_camera">
-                <update_rate>60</update_rate>
+                <update_rate>10</update_rate>
+                <topic>realsense</topic>
                 <camera name="camera">
                     <horizontal_fov>1.0472</horizontal_fov>
@@ -89,5 +74,5 @@
                         <clip>
                             <near>0.1</near>
-                            <far>10</far>
+                            <far>3</far>
                         </clip>
                     </depth_camera>
@@ -100,9 +85,9 @@
             </sensor>
         </gazebo>
-        <joint name="realsense_joint">
+        <joint name="realsense_joint" type="fixed">
             <child link="realsense_link" />
-            <parent link="$(base_link)" />
+            <parent link="${world_link_name}" />
+            <xacro:insert_block name="origin"/>
         </joint>
-    <
     </xacro:macro>
 </robot>
