Commit message: Experimented with mimic joints in Gazebo, but collisions aren't working. Rolling back to non-mimic gripper

File: src/bar_examples/maci/robot_description/maci.urdf.xacro (robot description, xacro)
@@ -38,8 +38,12 @@
         <xacro:ros2_position_controller joint_name="ur5_wrist_3_joint" />
         <xacro:ros2_position_controller joint_name="finger_joint" />
+        <xacro:ros2_position_controller joint_name="left_inner_finger_joint" />
+        <xacro:ros2_position_controller joint_name="right_outer_knuckle_joint" />
+        <xacro:ros2_position_controller joint_name="right_inner_finger_joint" />
     </ros2_control>
     <gazebo>
     <plugin filename="gz_ros2_control-system" name="gz_ros2_control::GazeboSimROS2ControlPlugin">
             <parameters>$(find maci)/config/ros2_control.yaml</parameters>
+            <hold_joints>True</hold_joints>
         </plugin>
     </gazebo>

File: src/bar_examples/robotiq_arg85_description/urdf/robotiq_arg2f.xacro (robot description, xacro)
@@ -11,5 +11,5 @@
         <origin xyz="0 0 0" rpy="0 0 0" />
         <geometry>
-          <mesh filename="package://robotiq_2f_140_gripper_visualization/meshes/visual/robotiq_arg2f_base_link.stl" />
+          <mesh filename="file://$(find robotiq_2f_140_gripper_visualization)/meshes/visual/robotiq_arg2f_base_link.stl" />
         </geometry>
         <material name="">
@@ -20,5 +20,5 @@
         <origin xyz="0 0 0" rpy="0 0 0" />
         <geometry>
-          <mesh filename="package://robotiq_2f_140_gripper_visualization/meshes/collision/robotiq_arg2f_base_link.stl" />
+          <mesh filename="file://$(find robotiq_2f_140_gripper_visualization)/meshes/collision/robotiq_arg2f_base_link.stl" />
         </geometry>
       </collision>
@@ -27,5 +27,4 @@
   <xacro:macro name="finger_joints" params="prefix fingerprefix reflect">
     <xacro:outer_finger_joint prefix="${prefix}" fingerprefix="${fingerprefix}"/>
-    <xacro:inner_knuckle_joint prefix="${prefix}" fingerprefix="${fingerprefix}" reflect="${reflect}"/>
     <xacro:inner_finger_joint prefix="${prefix}" fingerprefix="${fingerprefix}"/>
     <xacro:inner_finger_pad_joint prefix="${prefix}" fingerprefix="${fingerprefix}"/>
@@ -36,5 +35,4 @@
     <xacro:inner_finger prefix="${prefix}" fingerprefix="${fingerprefix}" stroke="${stroke}"/>
     <xacro:inner_finger_pad prefix="${prefix}" fingerprefix="${fingerprefix}"/>
-    <xacro:inner_knuckle prefix="${prefix}" fingerprefix="${fingerprefix}" stroke="${stroke}"/>
   </xacro:macro>
 </robot>

File: src/bar_examples/robotiq_arg85_description/urdf/robotiq_arg2f_140_model_macro.xacro (robot description, xacro)
@@ -7,16 +7,10 @@
         <origin xyz="-0.000200000000003065 0.0199435877845359 0.0292245259211331" rpy="0 0 0" />
         <mass value="0.00853198276973456" />
-        <inertia
-            ixx="2.89328108496468E-06"
-            ixy="-1.57935047237397E-19"
-            ixz="-1.93980378593255E-19"
-            iyy="1.86719750325683E-06"
-            iyz="-1.21858577871576E-06"
-            izz="1.21905238907251E-06" />
+        <inertia ixx="2.89328108496468E-06" ixy="-1.57935047237397E-19" ixz="-1.93980378593255E-19" iyy="1.86719750325683E-06" iyz="-1.21858577871576E-06" izz="1.21905238907251E-06" />
       </inertial>
       <visual>
         <origin xyz="0 0 0" rpy="0 0 0" />
         <geometry>
-          <mesh filename="package://robotiq_2f_140_gripper_visualization/meshes/visual/robotiq_arg2f_${stroke}_outer_knuckle.stl" />
+          <mesh filename="file://$(find robotiq_2f_140_gripper_visualization)/meshes/visual/robotiq_arg2f_${stroke}_outer_knuckle.stl" />
         </geometry>
         <material name="">
@@ -27,5 +21,5 @@
         <origin xyz="0 0 0" rpy="0 0 0" />
         <geometry>
-          <mesh filename="package://robotiq_2f_140_gripper_visualization/meshes/collision/robotiq_arg2f_${stroke}_outer_knuckle.stl" />
+          <mesh filename="file://$(find robotiq_2f_140_gripper_visualization)/meshes/collision/robotiq_arg2f_${stroke}_outer_knuckle.stl" />
         </geometry>
       </collision>
@@ -37,16 +31,10 @@
         <origin xyz="0.00030115855001899 0.0373907951953854 -0.0208027427000385" rpy="0 0 0" />
         <mass value="0.022614240507152" />
-        <inertia
-            ixx="1.52518312458174E-05"
-            ixy="9.76583423954399E-10"
-            ixz="-5.43838577022588E-10"
-            iyy="6.17694243867776E-06"
-            iyz="6.78636130740228E-06"
-            izz="1.16494917907219E-05" />
+        <inertia ixx="1.52518312458174E-05" ixy="9.76583423954399E-10" ixz="-5.43838577022588E-10" iyy="6.17694243867776E-06" iyz="6.78636130740228E-06" izz="1.16494917907219E-05" />
       </inertial>
       <visual>
         <origin xyz="0 0 0" rpy="0 0 0" />
         <geometry>
-          <mesh filename="package://robotiq_2f_140_gripper_visualization/meshes/visual/robotiq_arg2f_${stroke}_outer_finger.stl" />
+          <mesh filename="file://$(find robotiq_2f_140_gripper_visualization)/meshes/visual/robotiq_arg2f_${stroke}_outer_finger.stl" />
         </geometry>
         <material name="">
@@ -57,5 +45,5 @@
         <origin xyz="0 0 0" rpy="0 0 0" />
         <geometry>
-          <mesh filename="package://robotiq_2f_140_gripper_visualization/meshes/collision/robotiq_arg2f_${stroke}_outer_finger.stl" />
+          <mesh filename="file://$(find robotiq_2f_140_gripper_visualization)/meshes/collision/robotiq_arg2f_${stroke}_outer_finger.stl" />
         </geometry>
       </collision>
@@ -67,16 +55,10 @@
         <origin xyz="0.000123011831763771 0.0507850843201817 0.00103968640075166" rpy="0 0 0" />
         <mass value="0.0271177346495152" />
-        <inertia
-            ixx="2.61910379223783E-05"
-            ixy="-2.43616858946494E-07"
-            ixz="-6.37789906117123E-09"
-            iyy="2.8270243746167E-06"
-            iyz="-5.37200748039765E-07"
-            izz="2.83695868220296E-05" />
+        <inertia ixx="2.61910379223783E-05" ixy="-2.43616858946494E-07" ixz="-6.37789906117123E-09" iyy="2.8270243746167E-06" iyz="-5.37200748039765E-07" izz="2.83695868220296E-05" />
       </inertial>
       <visual>
         <origin xyz="0 0 0" rpy="0 0 0" />
         <geometry>
-          <mesh filename="package://robotiq_2f_140_gripper_visualization/meshes/visual/robotiq_arg2f_${stroke}_inner_knuckle.stl" />
+          <mesh filename="file://$(find robotiq_2f_140_gripper_visualization)/meshes/visual/robotiq_arg2f_${stroke}_inner_knuckle.stl" />
         </geometry>
         <material name="">
@@ -87,5 +69,5 @@
         <origin xyz="0 0 0" rpy="0 0 0" />
         <geometry>
-          <mesh filename="package://robotiq_2f_140_gripper_visualization/meshes/collision/robotiq_arg2f_${stroke}_inner_knuckle.stl" />
+          <mesh filename="file://$(find robotiq_2f_140_gripper_visualization)/meshes/collision/robotiq_arg2f_${stroke}_inner_knuckle.stl" />
         </geometry>
       </collision>
@@ -97,16 +79,10 @@
         <origin xyz="0.000299999999999317 0.0160078233491243 -0.0136945669206257" rpy="0 0 0" />
         <mass value="0.0104003125914103" />
-        <inertia
-            ixx="2.71909453810972E-06"
-            ixy="1.35402465472579E-21"
-            ixz="-7.1817349065269E-22"
-            iyy="7.69100314106116E-07"
-            iyz="6.74715432769696E-07"
-            izz="2.30315190420171E-06" />
+        <inertia ixx="2.71909453810972E-06" ixy="1.35402465472579E-21" ixz="-7.1817349065269E-22" iyy="7.69100314106116E-07" iyz="6.74715432769696E-07" izz="2.30315190420171E-06" />
       </inertial>
       <visual>
         <origin xyz="0 0 0" rpy="0 0 0" />
         <geometry>
-          <mesh filename="package://robotiq_2f_140_gripper_visualization/meshes/visual/robotiq_arg2f_${stroke}_inner_finger.stl" />
+          <mesh filename="file://$(find robotiq_2f_140_gripper_visualization)/meshes/visual/robotiq_arg2f_${stroke}_inner_finger.stl" />
         </geometry>
         <material name="">
@@ -117,5 +93,5 @@
         <origin xyz="0 0 0" rpy="0 0 0" />
         <geometry>
-          <mesh filename="package://robotiq_2f_140_gripper_visualization/meshes/collision/robotiq_arg2f_${stroke}_inner_finger.stl" />
+          <mesh filename="file://$(find robotiq_2f_140_gripper_visualization)/meshes/collision/robotiq_arg2f_${stroke}_inner_finger.stl" />
         </geometry>
       </collision>
@@ -137,5 +113,5 @@
         <origin xyz="0 0 0" rpy="0 0 0" />
         <geometry>
-           <box size="0.03 0.07 0.0075"/>
+          <box size="0.03 0.07 0.0075"/>
         </geometry>
         <material name="">
@@ -159,6 +135,6 @@
       <child link="${prefix}${fingerprefix}_inner_knuckle" />
       <axis xyz="1 0 0" />
-      <limit lower="-0.8757" upper="0.8757" velocity="2.0" effort="1000" />
-      <mimic joint="${prefix}finger_joint" multiplier="-1" offset="0" />
+      <limit lower="0" upper="0.8757" velocity="2.0" effort="1000" />
+      <!--  <mimic joint="${prefix}finger_joint" multiplier="-1" offset="0" /> -->
     </joint>
   </xacro:macro>
@@ -169,6 +145,6 @@
       <child link="${prefix}${fingerprefix}_inner_finger" />
       <axis xyz="1 0 0" />
-      <limit lower="-0.8757" upper="0.8757" velocity="2.0" effort="1000" />
-      <mimic joint="${prefix}finger_joint" multiplier="1" offset="0" />
+      <limit lower="0" upper="0.8757" velocity="2.0" effort="1000" />
+      <!--  <mimic joint="${prefix}finger_joint" multiplier="1" offset="0" /> -->
     </joint>
   </xacro:macro>
@@ -199,5 +175,5 @@
       <axis xyz="1 0 0" />
       <limit lower="-0.725" upper="0.725" velocity="2.0" effort="1000" />
-    <mimic joint="${prefix}finger_joint" multiplier="-1" offset="0" />
+      <!-- <mimic joint="${prefix}finger_joint" multiplier="-1" offset="0" /> -->
     </joint>
     <xacro:finger_joints prefix="${prefix}" fingerprefix="right" reflect="-1.0"/>

Commit message: Adding perception to Maci

File: src/bar_examples/maci/robot_description/maci.urdf.xacro (robot description, xacro)
@@ -1,13 +1,10 @@
 <?xml version='1.0' encoding='utf-8'?>
 <robot xmlns:xacro="http://www.ros.org/wiki/xacro" name="maci">
+    <xacro:include filename="$(find magni_description)/urdf/inertial.xacro" />
+    <xacro:include filename="$(find sensors)/realsense_d435/realsense.urdf.xacro" />
     <!-- Include a UR10 -->
     <xacro:include filename="$(find ur_description)/urdf/ur_macro.xacro" />
     <xacro:arg name="ur_type" default="ur5e"/>
-    <xacro:ur_robot name="ur5" tf_prefix="ur5_" parent="world"
-            joint_limits_parameters_file="$(find ur_description)/config/$(arg ur_type)/joint_limits.yaml"
-            kinematics_parameters_file="$(find ur_description)/config/$(arg ur_type)/default_kinematics.yaml"
-            physical_parameters_file="$(find ur_description)/config/$(arg ur_type)/physical_parameters.yaml"
-            visual_parameters_file="$(find ur_description)/config/$(arg ur_type)/visual_parameters.yaml"
-             >
+    <xacro:ur_robot name="ur5" tf_prefix="ur5_" parent="world" joint_limits_parameters_file="$(find ur_description)/config/$(arg ur_type)/joint_limits.yaml" kinematics_parameters_file="$(find ur_description)/config/$(arg ur_type)/default_kinematics.yaml" physical_parameters_file="$(find ur_description)/config/$(arg ur_type)/physical_parameters.yaml" visual_parameters_file="$(find ur_description)/config/$(arg ur_type)/visual_parameters.yaml">
         <origin xyz="-0.1 0 0.15" rpy="${pi} 0 0" />
     </xacro:ur_robot>
@@ -18,4 +15,8 @@
         <child link="robotiq_arg2f_base_link" />
     </joint>
+    <!-- Lets add a realsense camera to give some depth perception to Maci. -->
+    <xacro:realsense world_link_name="world">
+        <origin xyz="0 1.00 1.2" rpy="0 ${pi/4} -${pi/2}" />
+    </xacro:realsense>
     <xacro:macro name="ros2_position_controller" params="joint_name">
         <joint name="${joint_name}">
@@ -43,7 +44,9 @@
     </ros2_control>
     <gazebo>
-    <plugin filename="gz_ros2_control-system" name="gz_ros2_control::GazeboSimROS2ControlPlugin">
+        <plugin filename="gz_ros2_control-system" name="gz_ros2_control::GazeboSimROS2ControlPlugin">
             <parameters>$(find maci)/config/ros2_control.yaml</parameters>
-            <hold_joints>True</hold_joints>
+        </plugin>
+        <plugin filename="gz-sim-sensors-system" name="gz::sim::systems::Sensors">
+            <render_engine>ogre2</render_engine>
         </plugin>
     </gazebo>

File: src/bar_examples/sensors/realsense_d435/realsense.urdf.xacro (robot description, xacro)
@@ -5,4 +5,5 @@
             <xacro:box_inertial x="0.02" y="0.1" z="0.01" mass="0.06"/>
             <collision name="collision">
+                <origin rpy="0 0 ${pi/2}"/>
                 <geometry>
                     <mesh filename="package://sensors/realsense_d435/meshes/realsense.dae" />
