Commit message: Adjustments to get freecad to load krytn

File: src/bar_examples/krytn/robot_description/krytn.urdf.xacro (robot description, xacro)
@@ -1,4 +1,4 @@
 <?xml version='1.0' encoding='utf-8'?>
-<robot xmlns:xacro="http://www.ros.org/wiki/xacro" name="krytn">
+<robot xmlns:xacro="http://www.ros.org/wiki/xacro" name="krytn" encoding='UTF-8'>
   <!-- Import and add robot components -->
   <xacro:include filename="$(find magni_description)/urdf/magni.urdf.xacro" />

File: src/bar_examples/magni_description/urdf/inertial.xacro (robot description, xacro)
@@ -1,5 +1,5 @@
-<?xml version="1.0"?>
+<?xml version="1.0" ?>
 <!--
-Copyright 2019 Osnabrück University, Knowledge Based Systems Group
+Copyright 2019 Osnabruck University, Knowledge Based Systems Group
 https://github.com/uos/uos_tools/tree/kinetic/uos_common_urdf
 Redistribution and use in source and binary forms, with or without modification,
@@ -32,7 +32,5 @@
             <mass value="${mass}" />
             <origin xyz="0 0 0" />
-            <inertia ixx="${0.4 * mass * radius * radius}" ixy="0.0" ixz="0.0"
-                     iyy="${0.4 * mass * radius * radius}" iyz="0.0"
-                     izz="${0.4 * mass * radius * radius}" />
+            <inertia ixx="${0.4 * mass * radius * radius}" ixy="0.0" ixz="0.0" iyy="${0.4 * mass * radius * radius}" iyz="0.0" izz="${0.4 * mass * radius * radius}" />
         </inertial>
     </xacro:macro>
@@ -41,7 +39,5 @@
             <mass value="${mass}" />
             <origin xyz="0 0 0" />
-            <inertia ixx="${0.0833333 * mass * (3 * radius * radius + length * length)}" ixy="0.0" ixz="0.0"
-                     iyy="${0.0833333 * mass * (3 * radius * radius + length * length)}" iyz="0.0"
-                     izz="${0.5 * mass * radius * radius}" />
+            <inertia ixx="${0.0833333 * mass * (3 * radius * radius + length * length)}" ixy="0.0" ixz="0.0" iyy="${0.0833333 * mass * (3 * radius * radius + length * length)}" iyz="0.0" izz="${0.5 * mass * radius * radius}" />
         </inertial>
     </xacro:macro>
@@ -50,7 +46,5 @@
             <mass value="${mass}" />
             <origin xyz="-0.15 0 0.03" />
-            <inertia ixx="${0.0833333 * mass * (y*y + z*z)}" ixy="0.0" ixz="0.0"
-                     iyy="${0.0833333 * mass * (x*x + z*z)}" iyz="0.0"
-                     izz="${0.0833333 * mass * (x*x + y*y)}" />
+            <inertia ixx="${0.0833333 * mass * (y*y + z*z)}" ixy="0.0" ixz="0.0" iyy="${0.0833333 * mass * (x*x + z*z)}" iyz="0.0" izz="${0.0833333 * mass * (x*x + y*y)}" />
         </inertial>
     </xacro:macro>
@@ -60,7 +54,5 @@
             <mass value="${mass}" />
             <xacro:insert_block name="origin" />
-            <inertia ixx="${0.4 * mass * radius * radius}" ixy="0.0" ixz="0.0"
-                     iyy="${0.4 * mass * radius * radius}" iyz="0.0"
-                     izz="${0.4 * mass * radius * radius}" />
+            <inertia ixx="${0.4 * mass * radius * radius}" ixy="0.0" ixz="0.0" iyy="${0.4 * mass * radius * radius}" iyz="0.0" izz="${0.4 * mass * radius * radius}" />
         </inertial>
     </xacro:macro>
@@ -69,7 +61,5 @@
             <mass value="${mass}" />
             <xacro:insert_block name="origin" />
-            <inertia ixx="${0.0833333 * mass * (3 * radius * radius + length * length)}" ixy="0.0" ixz="0.0"
-                     iyy="${0.0833333 * mass * (3 * radius * radius + length * length)}" iyz="0.0"
-                     izz="${0.5 * mass * radius * radius}" />
+            <inertia ixx="${0.0833333 * mass * (3 * radius * radius + length * length)}" ixy="0.0" ixz="0.0" iyy="${0.0833333 * mass * (3 * radius * radius + length * length)}" iyz="0.0" izz="${0.5 * mass * radius * radius}" />
         </inertial>
     </xacro:macro>
@@ -78,7 +68,5 @@
             <mass value="${mass}" />
             <xacro:insert_block name="origin" />
-            <inertia ixx="${0.0833333 * mass * (y*y + z*z)}" ixy="0.0" ixz="0.0"
-                     iyy="${0.0833333 * mass * (x*x + z*z)}" iyz="0.0"
-                     izz="${0.0833333 * mass * (x*x + y*y)}" />
+            <inertia ixx="${0.0833333 * mass * (y*y + z*z)}" ixy="0.0" ixz="0.0" iyy="${0.0833333 * mass * (x*x + z*z)}" iyz="0.0" izz="${0.0833333 * mass * (x*x + y*y)}" />
         </inertial>
     </xacro:macro>

File: src/bar_examples/magni_description/urdf/magni.urdf.xacro (robot description, xacro)
@@ -1,3 +1,3 @@
-<?xml version="1.0"?>
+<?xml version="1.0" encoding='UTF-8'?>
 <robot xmlns:xacro="http://www.ros.org/wiki/xacro">
   <xacro:property name="wheel_r" value="0.1" />
@@ -106,5 +106,5 @@
       <origin xyz="0 ${0.163*reflect} 0" rpy="0 0 ${pi/2}"/>
       <dynamics damping="0.2" friction="0.8"/>
-      <limit effort="1000" velocity="10" stiffness="0" dissipation="0"/>
+      <limit effort="1000" velocity="10"/>
     </joint>
     <gazebo reference="${prefix}_wheel">

Commit message: Initial commit

File: src/bar_examples/krytn/robot_description/krytn.urdf.xacro (robot description, xacro)
@@ -11,4 +11,28 @@
     <origin xyz="0 0 0.15" rpy="0 0 0" />
   </xacro:lidar_2d>
+  <link name="krtyn_tray">
+    <visual>
+      <!--Part/Body.-->
+      <origin rpy="0.0 -0.0 0.0" xyz="0.0 0.0 0.0"/>
+      <geometry>
+        <mesh filename="package://kyrtyn_tray/meshes/Krtyn_Tray_Ex2_Body.dae"/>
+      </geometry>
+    </visual>
+    <collision>
+      <!--Part/Body.-->
+      <origin rpy="0.0 -0.0 0.0" xyz="0.0 0.0 0.0"/>
+      <geometry>
+        <mesh filename="package://kyrtyn_tray/meshes/Krtyn_Tray_Ex2_Body.dae"/>
+      </geometry>
+    </collision>
+    <xacro:box_inertial_with_origin x="0.398" y="0.221" z="0.150" mass="1.0">
+      <origin xyz="-0.0 0 0" rpy="0 0 0" />
+    </xacro:box_inertial_with_origin>
+  </link>
+  <joint name="tray_joint" type="fixed">
+    <parent link="base_link"/>
+    <child link="krtyn_tray"/>
+    <origin rpy="0.0 -0.0 3.141592653589793" xyz="-0.09 -0.17 0.165"/>
+  </joint>
   <!-- Configure Control of Joints -->
   <ros2_control name="Krytn" type="system">
