Commit message: Initial commit

File: src/my_robot_arm/urdf/my_robot_arm.urdf.xacro (robot description, xacro)
@@ -3,4 +3,5 @@
     <xacro:include filename="$(find magni_description)/urdf/inertial.xacro" />
     <xacro:property name="initial_positions" value="${load_yaml(find(my_robot_arm)/config)['initial_positions']}"/>
+    <xacro:include filename="$(find sensors)/realsense_d435/realsense.urdf.xacro" />
     <!-- Include a UR5 -->
     <xacro:include filename="$(find ur_description)/urdf/ur_macro.xacro" />
@@ -10,4 +11,7 @@
     </xacro:ur_robot>
     <link name="world" />
+    <xacro:realsense world_link_name="world">
+        <origin xyz="0 4.0 4.2" rpy="0 ${pi/4} -${pi/2}" />
+    </xacro:realsense>
     <link name="base_link">
         <visual>
