Commit message: Adding big collision cylinders to new wheels

File: src/security_robot_freecad/urdf/FirstRobot.urdf (robot description, URDF)
Before this commit: robot Robot, 7 links, 6 joints
Links:
- link Front_Left_Wheel: mass 0.0 -> 0.7509245446194294; geometry collision cylinder length=0.03000000000000005 radius=0.06; visual mesh filename=package://security_robot_freecad/meshes/first_robot_Securit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
- link Front_Right_Wheel: mass 0.0 -> 0.7509245446194294; geometry collision cylinder length=0.03000000000000005 radius=0.06; visual mesh filename=package://security_robot_freecad/meshes/first_robot_Securit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

Commit message: increase diameter of collision cylinder.

File: src/security_robot_freecad/urdf/FirstRobot.urdf (robot description, URDF)
Before this commit: robot Robot, 7 links, 6 joints
Links:
- link Front_Left_Wheel: geometry collision cylinder length=0.03000000000000005 radius=0.3; visual mesh filename=package://security_robot_freecad/meshes/first_robot_Securit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
- link Front_Right_Wheel: geometry collision cylinder length=0.03000000000000005 radius=0.3; visual mesh filename=package://security_robot_freecad/meshes/first_robot_Securit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
- link Sensor_Link_01: geometry collision cylinder length=0.03000000000000005 radius=0.3; visual mesh filename=package://security_robot_freecad/meshes/first_robot_Securit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
- link left_wheel: geometry collision cylinder length=0.03000000000000005 radius=0.3; visual mesh filename=package://security_robot_freecad/meshes/first_robot_Securit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
- link right_wheel: geometry collision cylinder length=0.03000000000000005 radius=0.3; visual mesh filename=package://security_robot_freecad/meshes/first_robot_Securit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

Commit message: Initial commit

File: src/security_robot_freecad/urdf/FirstRobot.urdf (robot description, URDF)
Before this commit: robot Robot, 7 links, 6 joints
Links:
- link Front_Left_Wheel: mass 0.0 -> 0.7509245446194294
- link Front_Right_Wheel: mass 0.0 -> 0.7509245446194294
- link base_link: mass 6.4799999999999995 -> 1.4799999999999995
- link left_wheel: geometry collision mesh filename=package://security_robot_freecad/meshes/first_robot_Securit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; visual mesh filename=package://security_robot_freecad/meshes/first_robot_Securit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
- link right_wheel: geometry collision mesh filename=package://security_robot_freecad/meshes/first_robot_Securit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; visual mesh filename=package://security_robot_freecad/meshes/first_robot_Securit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
Joints:
- joint Front_Left_Wheel_Joint: axis (none) -> 0 0 1; origin xyz=-1.7 0.25 -0.37 rpy=-1.5707963267948966 0.0 0.0 -> xyz=-1.7 0.25 -0.257 rpy=-1.5707963267948966 0.0 0.0
- joint Front_Right_Wheel_Joint: axis (none) -> 0 0 1; origin xyz=-1.7 -0.25 -0.37 rpy=-1.5707963267948966 0.0 0.0 -> xyz=-1.7 -0.25 -0.257 rpy=-1.5707963267948966 0.0 0.0
- joint left_wheel_joint: origin xyz=-0.355 0.25 -0.35 rpy=-1.5707963267948966 0.0 0.0 -> xyz=-0.355 0.25 -0.255 rpy=-1.5707963267948966 0.0 0.0
- joint right_wheel_joint: origin xyz=-0.355 -0.25 -0.35 rpy=-1.5707963267948966 0.0 0.0 -> xyz=-0.355 -0.25 -0.255 rpy=-1.5707963267948966 0.0 0.0
